Commit message: added all urdfs to package

File: urdf/coupling1.urdf.xacro (robot description, xacro)
@@ -4,21 +4,21 @@
      For more information, please see http://wiki.ros.org/sw_urdf_exporter -->
 <robot
-  name="probe_mount2"
+  name="coupling1"
   xmlns:xacro="http://www.ros.org/wiki/xacro">
   <link
-    name="link_probe">
+    name="link_coupling1">
     <inertial>
       <origin
-        xyz="0.0172095025438958 -0.0934181562801906 0.000471391183381434"
+        xyz="1.77823331599424E-05 -1.77823331599619E-05 -0.0089016237884829"
         rpy="0 0 0" />
       <mass
-        value="0.275178819498116" />
+        value="0.0748232729606399" />
       <inertia
-        ixx="0.00158144645389415"
-        ixy="9.09904679448213E-05"
-        ixz="-2.74539325678678E-06"
-        iyy="0.000168425924534353"
-        iyz="3.76040071661897E-05"
-        izz="0.00150104046709865" />
+        ixx="3.39450510121467E-05"
+        ixy="4.13727922672199E-08"
+        ixz="-8.51756765772707E-09"
+        iyy="3.39450510121467E-05"
+        iyz="8.51756765772627E-09"
+        izz="5.88806034471799E-05" />
     </inertial>
     <visual>
@@ -28,10 +28,10 @@
       <geometry>
         <mesh
-          filename="package://system_urdf/meshes/probe_mount/probe_mount.STL" />
+          filename="package://system_urdf/meshes/roller_probe_pieces/coupling1.STL" />
       </geometry>
       <material
         name="">
         <color
-          rgba="0.0196078431372549 0.0196078431372549 0.0196078431372549 1" />
+          rgba="0.749019607843137 0.749019607843137 0.749019607843137 1" />
       </material>
     </visual>
@@ -42,5 +42,5 @@
       <geometry>
         <mesh
-          filename="package://system_urdf/meshes/probe_mount/probe_mount.STL" />
+          filename="package://system_urdf/meshes/roller_probe_pieces/coupling1.STL" />
       </geometry>
     </collision>

File: urdf/coupling2.urdf.xacro (robot description, xacro)
@@ -4,21 +4,21 @@
      For more information, please see http://wiki.ros.org/sw_urdf_exporter -->
 <robot
-  name="probe_mount2"
+  name="coupling2"
   xmlns:xacro="http://www.ros.org/wiki/xacro">
   <link
-    name="link_probe">
+    name="link_coupling2">
     <inertial>
       <origin
-        xyz="0.0172095025438958 -0.0934181562801906 0.000471391183381434"
+        xyz="5.88703171151242E-05 -8.94009617138191E-05 -0.00263303385335754"
         rpy="0 0 0" />
       <mass
-        value="0.275178819498116" />
+        value="0.0395051823054991" />
       <inertia
-        ixx="0.00158144645389415"
-        ixy="9.09904679448213E-05"
-        ixz="-2.74539325678678E-06"
-        iyy="0.000168425924534353"
-        iyz="3.76040071661897E-05"
-        izz="0.00150104046709865" />
+        ixx="2.30288040660326E-05"
+        ixy="7.2150343292927E-08"
+        ixz="-6.58246910799801E-10"
+        iyy="2.3069990933938E-05"
+        iyz="9.99619328617187E-10"
+        izz="4.59060223616661E-05" />
     </inertial>
     <visual>
@@ -28,10 +28,10 @@
       <geometry>
         <mesh
-          filename="package://system_urdf/meshes/probe_mount/probe_mount.STL" />
+          filename="package://system_urdf/meshes/roller_probe_pieces/coupling2.STL" />
       </geometry>
       <material
         name="">
         <color
-          rgba="0.0196078431372549 0.0196078431372549 0.0196078431372549 1" />
+          rgba="0.749019607843137 0.749019607843137 0.749019607843137 1" />
       </material>
     </visual>
@@ -42,5 +42,5 @@
       <geometry>
         <mesh
-          filename="package://system_urdf/meshes/probe_mount/probe_mount.STL" />
+          filename="package://system_urdf/meshes/roller_probe_pieces/coupling2.STL" />
       </geometry>
     </collision>

File: urdf/coupling3.urdf.xacro (robot description, xacro)
@@ -4,21 +4,21 @@
      For more information, please see http://wiki.ros.org/sw_urdf_exporter -->
 <robot
-  name="probe_mount2"
+  name="ee"
   xmlns:xacro="http://www.ros.org/wiki/xacro">
   <link
-    name="link_probe">
+    name="link_coupling3">
     <inertial>
       <origin
-        xyz="0.0172095025438958 -0.0934181562801906 0.000471391183381434"
+        xyz="-2.13510948500582E-07 -1.82970595220083E-06 -0.00768363431196126"
         rpy="0 0 0" />
       <mass
-        value="0.275178819498116" />
+        value="0.0384214421870518" />
       <inertia
-        ixx="0.00158144645389415"
-        ixy="9.09904679448213E-05"
-        ixz="-2.74539325678678E-06"
-        iyy="0.000168425924534353"
-        iyz="3.76040071661897E-05"
-        izz="0.00150104046709865" />
+        ixx="1.44308944749129E-05"
+        ixy="1.10001208358471E-10"
+        ixz="6.16955726898917E-11"
+        iyy="1.44318430502768E-05"
+        iyz="5.28407477246946E-10"
+        izz="2.80517055222733E-05" />
     </inertial>
     <visual>
@@ -28,10 +28,10 @@
       <geometry>
         <mesh
-          filename="package://system_urdf/meshes/probe_mount/probe_mount.STL" />
+          filename="package://system_urdf/meshes/roller_probe_pieces/coupling3.STL" />
       </geometry>
       <material
         name="">
         <color
-          rgba="0.0196078431372549 0.0196078431372549 0.0196078431372549 1" />
+          rgba="0.749019607843137 0.749019607843137 0.749019607843137 1" />
       </material>
     </visual>
@@ -42,5 +42,5 @@
       <geometry>
         <mesh
-          filename="package://system_urdf/meshes/probe_mount/probe_mount.STL" />
+          filename="package://system_urdf/meshes/roller_probe_pieces/coupling3.STL" />
       </geometry>
     </collision>

File: urdf/extender.urdf.xacro (robot description, xacro)
@@ -3,22 +3,21 @@
      Commit Version: 1.6.0-4-g7f85cfe  Build Version: 1.6.7995.38578
      For more information, please see http://wiki.ros.org/sw_urdf_exporter -->
-<robot
-  name="probe_mount2"
-  xmlns:xacro="http://www.ros.org/wiki/xacro">
+<robot xmlns:xacro="http://www.ros.org/wiki/xacro"
+  name="extender">
   <link
-    name="link_probe">
+    name="link_extender">
     <inertial>
       <origin
-        xyz="0.0172095025438958 -0.0934181562801906 0.000471391183381434"
+        xyz="-5.17709074753684E-17 2.39346204362228E-17 0.023707057889378"
         rpy="0 0 0" />
       <mass
-        value="0.275178819498116" />
+        value="0.0901411341968167" />
       <inertia
-        ixx="0.00158144645389415"
-        ixy="9.09904679448213E-05"
-        ixz="-2.74539325678678E-06"
-        iyy="0.000168425924534353"
-        iyz="3.76040071661897E-05"
-        izz="0.00150104046709865" />
+        ixx="3.21898550179311E-05"
+        ixy="2.53970297447911E-21"
+        ixz="3.5531232175751E-20"
+        iyy="3.21898550179311E-05"
+        iyz="-1.94420820770643E-20"
+        izz="2.82781083124868E-05" />
     </inertial>
     <visual>
@@ -28,10 +27,10 @@
       <geometry>
         <mesh
-          filename="package://system_urdf/meshes/probe_mount/probe_mount.STL" />
+          filename="package://system_urdf/meshes/roller_probe_pieces/extender.STL" />
       </geometry>
       <material
         name="">
         <color
-          rgba="0.0196078431372549 0.0196078431372549 0.0196078431372549 1" />
+          rgba="0.749019607843137 0.749019607843137 0.749019607843137 1" />
       </material>
     </visual>
@@ -42,5 +41,5 @@
       <geometry>
         <mesh
-          filename="package://system_urdf/meshes/probe_mount/probe_mount.STL" />
+          filename="package://system_urdf/meshes/roller_probe_pieces/extender.STL" />
       </geometry>
     </collision>

File: urdf/ft_sensor.urdf.xacro (robot description, xacro)
@@ -4,21 +4,21 @@
      For more information, please see http://wiki.ros.org/sw_urdf_exporter -->
 <robot
-  name="probe_mount2"
+  name="ft_sensor"
   xmlns:xacro="http://www.ros.org/wiki/xacro">
   <link
-    name="link_probe">
+    name="link_ft_sensor">
     <inertial>
       <origin
-        xyz="0.0172095025438958 -0.0934181562801906 0.000471391183381434"
+        xyz="-0.00152921654106877 0.00302047148579856 -0.0158969383860535"
         rpy="0 0 0" />
       <mass
-        value="0.275178819498116" />
+        value="0.00405727824464069" />
       <inertia
-        ixx="0.00158144645389415"
-        ixy="9.09904679448213E-05"
-        ixz="-2.74539325678678E-06"
-        iyy="0.000168425924534353"
-        iyz="3.76040071661897E-05"
-        izz="0.00150104046709865" />
+        ixx="2.11438887462202E-06"
+        ixy="1.86490444186628E-07"
+        ixz="4.91600397505994E-09"
+        iyy="1.82605884169168E-06"
+        iyz="-2.43792170617711E-08"
+        izz="3.23118515297441E-06" />
     </inertial>
     <visual>
@@ -28,10 +28,10 @@
       <geometry>
         <mesh
-          filename="package://system_urdf/meshes/probe_mount/probe_mount.STL" />
+          filename="package://system_urdf/meshes/roller_probe_pieces/ft_sensor.STL" />
       </geometry>
       <material
         name="">
         <color
-          rgba="0.0196078431372549 0.0196078431372549 0.0196078431372549 1" />
+          rgba="0.752941176470588 0.752941176470588 0.752941176470588 1" />
       </material>
     </visual>
@@ -42,5 +42,5 @@
       <geometry>
         <mesh
-          filename="package://system_urdf/meshes/probe_mount/probe_mount.STL" />
+          filename="package://system_urdf/meshes/roller_probe_pieces/ft_sensor.STL" />
       </geometry>
     </collision>

File: urdf/system.urdf.xacro (robot description, xacro)
@@ -15,13 +15,11 @@
     <xacro:include filename="kr10_r1100_2_urdf.urdf.xacro" />
     <!-- Import the ut horizontal end effector xacro model -->
-    <xacro:include filename="$(find probe_mount2)/urdf/probe_mount2.urdf.xacro"/>
-    <!-- Import the first coupling plate xacro -->
-    <!-- <xacro:include filename="$(find coupling1_urdf)/urdf/coupling1.urdf.xacro"/> -->
-    <!-- Import the ft sensor xacro -->
-    <!-- <xacro:include filename="$(find ft_sensor_urdf)/urdf/ft_sensor.urdf.xacro"/> -->
-    <!-- Import the second coupling plate xacro -->
-    <!-- <xacro:include filename="$(find coupling2_urdf)/urdf/coupling2.urdf.xacro"/> -->
-    <!-- Import the third coupling plate xacro -->
-    <!-- <xacro:include filename="$(find ee_urdf)/urdf/coupling3.urdf.xacro"/> -->
+    <xacro:include filename="probe_mount2.urdf.xacro"/>
+    <!-- Import the roller probe components xacro (separated to allow removal of any piece) -->
+    <xacro:include filename="coupling1.urdf.xacro"/>
+    <xacro:include filename="ft_sensor.urdf.xacro"/>
+    <xacro:include filename="coupling2.urdf.xacro"/>
+    <xacro:include filename="coupling3.urdf.xacro"/>
+    <xacro:include filename="extender.urdf.xacro" />
     <!-- ====================================================================================== -->
                                <!-- Add the tool center point  -->
@@ -47,36 +45,42 @@
     <!-- connect the pieces -->
     <!-- ========================================================================================= -->
-    <!--                                Beginning of 7.14 Configuration                            -->
+    <!--                   Beginning of extra  roller probe pieces Configuration                   -->
     <!-- ========================================================================================= -->
     <!-- kr10 to first coupling plate connection-->
-<!--     <joint name="kr10_coupling1_joint" type="fixed">
+    <joint name="kr10_coupling1_joint" type="fixed">
         <parent link="link_6"/>
         <child link="link_coupling1"/>
         <origin xyz="0 0 .02" rpy="${-pi/2} 0 0"/>
-    </joint>  -->
-    <!-- kr10 to end_effector connection-->
-<!--     <joint name="coupling1_coupling2" type="fixed">
+    </joint>
+    <!-- first coupling plate to ft_sensor-->
+    <joint name="coupling1_coupling2" type="fixed">
         <parent link="link_coupling1"/>
         <child link="link_coupling2"/>
         <origin xyz="0 0.005 0" rpy="0 0 0"/>
-    </joint>  -->
-    <!-- kr10 to end_effector connection-->
-<!--     <joint name="coupling2_ft_joint" type="fixed">
+    </joint>
+    <!-- ft_sensor to coupling plate 2-->
+    <joint name="coupling2_ft_joint" type="fixed">
         <parent link="link_coupling2"/>
-        <child link="ft_sensor"/>
+        <child link="link_ft_sensor"/>
         <origin xyz="0 0 0" rpy="${-pi} 0 0"/>
-    </joint>  -->
-    <!-- plate 3 to end_effector connection-->
-<!--     <joint name="kr10_endeffector_joint" type="fixed">
-        <parent link="ft_sensor"/>
-        <child link="link_ee"/>
+    </joint>
+    <!-- coupling plate 2 to end effector connection-->
+    <joint name="ft_coupling3_joint" type="fixed">
+        <parent link="link_ft_sensor"/>
+        <child link="link_coupling3"/>
         <origin xyz="0 0.0435 0" rpy="${pi} 0 0"/>
-    </joint>  -->
-    <!-- kr10 to end_effector connection-->
-<!--     <joint name="endeffector_utprobe_joint" type="fixed">
-        <parent link="link_ee"/>
-        <child link="probe_mount"/>
-        <origin xyz="0 0 0" rpy="${-pi/2} ${-pi/2} 0"/>
-    </joint>  -->
+    </joint>
+    <!-- coupling3 to extender connection-->
+    <joint name="coupling3_extender_joint" type="fixed">
+        <parent link="link_coupling3"/>
+        <child link="link_extender"/>
+        <origin xyz="0 0 0" rpy="0 0 0"/>
+    </joint>
+    <!-- -->
+    <joint name="extender_probe_joint" type="fixed">
+        <parent link="link_extender"/>
+        <child link="link_probe"/>
+        <origin xyz="0 -0.05 0" rpy="${-pi/2} ${-pi/2} 0"/>
+    </joint>
     <!-- ========================================================================================= -->
     <!--                                   End of 7.14 Configuration                               -->
@@ -86,22 +90,16 @@
     <!-- ========================================================================================= -->
 <!-- kr10 to Probe mount -->
+<!--
     <joint name="link_6_ut_probe_joint" type="fixed">
       <parent link="link_6"/>
       <child link="probe_mount"/>
       <origin xyz="0 0 0" rpy="${pi} 0 0"/>
-    </joint>
+    </joint> -->
     <!-- ========================================================================================= -->
     <!--                                       Same for Both                                       -->
     <!-- ========================================================================================= -->
-    <!-- end_effector to TCP for whole system -->
-<!--     <joint name="tool_center_joint" type="fixed">
-      <parent link="probe_mount"/>
-      <child link="tool_center_point"/>
-      <origin xyz="0.0125 ${-(n_focals * element_pitch / (2 * 1000)) + (64 * element_pitch / (2 *1000))} -0.245" rpy="${pi} 0 ${pi/2}"/>
-    </joint>
- -->
     <!-- end_effector to TCP -->
     <joint name="tool_center_joint" type="fixed">
-      <parent link="probe_mount"/>
+      <parent link="link_probe"/>
       <child link="tool_center_point"/>
       <origin xyz="0.0125 ${-(n_focals * element_pitch / (2 * 1000)) + (64 * element_pitch / (2 *1000))} -0.245" rpy="${pi} 0 ${pi/2}"/>
